File: glr-pcb-brake-light.kicad_sch (KiCad schematic)
At the start: 31 parts

Commit message: überarbeitung pcb, sch mit stecker
Parts:
- removed TP1, TP2: TestPoint, TestPoint:TestPoint_Keystone_5010-5014_Multipurpose, symbol Connector:TestPoint
- added J1: Conn_01x04_Pin, GLR_KiCad_Library:Wuerth_M12-Right-Angled-THT, symbol Connector:Conn_01x04_Pin
Connections:
- net GND: now reaches D12.1 (K), D18.1 (K), D24.1 (K), D6.1 (K)
- net GND: now also J1.2 (Pin_2)
- net +24V: now reaches D25.2 (A)
- net +24V: now also J1.1 (Pin_1)
- no-connect marks 0 -> 2

Commit message: pcb umdesigned fast fertig
Parts:
- J1: footprint GLR_KiCad_Library:Wuerth_M12-Right-Angled-THT -> GLR_KiCad_Library:Wuerth_M12-Panel-Cut-THT
Changed lines of the file:
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@@
 			)
 		)
-		(property "Footprint" "GLR_KiCad_Library:Wuerth_M12-Right-Angled-THT"
+		(property "Footprint" "GLR_KiCad_Library:Wuerth_M12-Panel-Cut-THT"
 			(at 34.29 27.94 0)
 			(hide yes)

Commit message: teile auf rückseite gebracht
Parts:
- D1, D10, D11, D12, D13, D14, D15, D16, D17, D18, D19, D2, D20, D21, D22, D23, D24, D3, D4, D5, D6, D7, D8, D9: footprint LED_SMD:LED_Avago_PLCC4_3.2x2.8mm_CW -> GLR_KiCad_Library:LED_Avago_PLCC4_3.2x2.8mm_CW
Changed lines of the file:
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@@
 			)
 		)
-		(property "Footprint" "LED_SMD:LED_Avago_PLCC4_3.2x2.8mm_CW"
+		(property "Footprint" "GLR_KiCad_Library:LED_Avago_PLCC4_3.2x2.8mm_CW"
 			(at 88.9 66.04 0)
 			(hide yes)
@@
 			)
 		)
-		(property "Footprint" "LED_SMD:LED_Avago_PLCC4_3.2x2.8mm_CW"
+		(property "Footprint" "GLR_KiCad_Library:LED_Avago_PLCC4_3.2x2.8mm_CW"
 			(at 107.95 96.52 0)
 			(hide yes)
@@
 			)
 		)
-		(property "Footprint" "LED_SMD:LED_Avago_PLCC4_3.2x2.8mm_CW"
+		(property "Footprint" "GLR_KiCad_Library:LED_Avago_PLCC4_3.2x2.8mm_CW"
 			(at 107.95 81.28 0)
 			(hide yes)
@@
 			)
 		)
-		(property "Footprint" "LED_SMD:LED_Avago_PLCC4_3.2x2.8mm_CW"
+		(property "Footprint" "GLR_KiCad_Library:LED_Avago_PLCC4_3.2x2.8mm_CW"
 			(at 107.95 110.49 0)
 			(hide yes)
@@
 			)
 		)
-		(property "Footprint" "LED_SMD:LED_Avago_PLCC4_3.2x2.8mm_CW"
+		(property "Footprint" "GLR_KiCad_Library:LED_Avago_PLCC4_3.2x2.8mm_CW"
 			(at 125.73 125.73 0)
 			(hide yes)
@@
 			)
 		)
-		(property "Footprint" "LED_SMD:LED_Avago_PLCC4_3.2x2.8mm_CW"
+		(property "Footprint" "GLR_KiCad_Library:LED_Avago_PLCC4_3.2x2.8mm_CW"
 			(at 125.73 66.04 0)
 			(hide yes)
@@
 			)
 		)
-		(property "Footprint" "LED_SMD:LED_Avago_PLCC4_3.2x2.8mm_CW"
+		(property "Footprint" "GLR_KiCad_Library:LED_Avago_PLCC4_3.2x2.8mm_CW"
 			(at 69.85 125.73 0)
 			(hide yes)
@@
 			)
 		)
-		(property "Footprint" "LED_SMD:LED_Avago_PLCC4_3.2x2.8mm_CW"
+		(property "Footprint" "GLR_KiCad_Library:LED_Avago_PLCC4_3.2x2.8mm_CW"
 			(at 125.73 52.07 0)
 			(hide yes)
@@
 			)
 		)
-		(property "Footprint" "LED_SMD:LED_Avago_PLCC4_3.2x2.8mm_CW"
+		(property "Footprint" "GLR_KiCad_Library:LED_Avago_PLCC4_3.2x2.8mm_CW"
 			(at 88.9 81.28 0)
 			(hide yes)
@@
 			)
 		)
-		(property "Footprint" "LED_SMD:LED_Avago_PLCC4_3.2x2.8mm_CW"
+		(property "Footprint" "GLR_KiCad_Library:LED_Avago_PLCC4_3.2x2.8mm_CW"
 			(at 125.73 96.52 0)
 			(hide yes)
@@
 			)
 		)
-		(property "Footprint" "LED_SMD:LED_Avago_PLCC4_3.2x2.8mm_CW"
+		(property "Footprint" "GLR_KiCad_Library:LED_Avago_PLCC4_3.2x2.8mm_CW"
 			(at 69.85 96.52 0)
 			(hide yes)
@@
 			)
 		)
-		(property "Footprint" "LED_SMD:LED_Avago_PLCC4_3.2x2.8mm_CW"
+		(property "Footprint" "GLR_KiCad_Library:LED_Avago_PLCC4_3.2x2.8mm_CW"
 			(at 69.85 52.07 0)
 			(hide yes)
@@
 			)
 		)
-		(property "Footprint" "LED_SMD:LED_Avago_PLCC4_3.2x2.8mm_CW"
+		(property "Footprint" "GLR_KiCad_Library:LED_Avago_PLCC4_3.2x2.8mm_CW"
 			(at 107.95 125.73 0)
 			(hide yes)
@@
 			)
 		)
-		(property "Footprint" "LED_SMD:LED_Avago_PLCC4_3.2x2.8mm_CW"
+		(property "Footprint" "GLR_KiCad_Library:LED_Avago_PLCC4_3.2x2.8mm_CW"
 			(at 88.9 110.49 0)
 			(hide yes)
@@
 			)
 		)
-		(property "Footprint" "LED_SMD:LED_Avago_PLCC4_3.2x2.8mm_CW"
+		(property "Footprint" "GLR_KiCad_Library:LED_Avago_PLCC4_3.2x2.8mm_CW"
 			(at 125.73 110.49 0)
 			(hide yes)
@@
 			)
 		)
-		(property "Footprint" "LED_SMD:LED_Avago_PLCC4_3.2x2.8mm_CW"
+		(property "Footprint" "GLR_KiCad_Library:LED_Avago_PLCC4_3.2x2.8mm_CW"
 			(at 88.9 125.73 0)
 			(hide yes)
@@
 			)
 		)
-		(property "Footprint" "LED_SMD:LED_Avago_PLCC4_3.2x2.8mm_CW"
+		(property "Footprint" "GLR_KiCad_Library:LED_Avago_PLCC4_3.2x2.8mm_CW"
 			(at 125.73 81.28 0)
 			(hide yes)
@@
 			)
 		)
-		(property "Footprint" "LED_SMD:LED_Avago_PLCC4_3.2x2.8mm_CW"
+		(property "Footprint" "GLR_KiCad_Library:LED_Avago_PLCC4_3.2x2.8mm_CW"
 			(at 88.9 52.07 0)
 			(hide yes)
@@
 			)
 		)
-		(property "Footprint" "LED_SMD:LED_Avago_PLCC4_3.2x2.8mm_CW"
+		(property "Footprint" "GLR_KiCad_Library:LED_Avago_PLCC4_3.2x2.8mm_CW"
 			(at 107.95 66.04 0)
 			(hide yes)
@@
 			)
 		)
-		(property "Footprint" "LED_SMD:LED_Avago_PLCC4_3.2x2.8mm_CW"
+		(property "Footprint" "GLR_KiCad_Library:LED_Avago_PLCC4_3.2x2.8mm_CW"
 			(at 69.85 66.04 0)
 			(hide yes)
@@
 			)
 		)
-		(property "Footprint" "LED_SMD:LED_Avago_PLCC4_3.2x2.8mm_CW"
+		(property "Footprint" "GLR_KiCad_Library:LED_Avago_PLCC4_3.2x2.8mm_CW"
 			(at 88.9 96.52 0)
 			(hide yes)
@@
 			)
 		)
-		(property "Footprint" "LED_SMD:LED_Avago_PLCC4_3.2x2.8mm_CW"
+		(property "Footprint" "GLR_KiCad_Library:LED_Avago_PLCC4_3.2x2.8mm_CW"
 			(at 107.95 52.07 0)
 			(hide yes)
@@
 			)
 		)
-		(property "Footprint" "LED_SMD:LED_Avago_PLCC4_3.2x2.8mm_CW"
+		(property "Footprint" "GLR_KiCad_Library:LED_Avago_PLCC4_3.2x2.8mm_CW"
 			(at 69.85 81.28 0)
 			(hide yes)
@@
 			)
 		)
-		(property "Footprint" "LED_SMD:LED_Avago_PLCC4_3.2x2.8mm_CW"
+		(property "Footprint" "GLR_KiCad_Library:LED_Avago_PLCC4_3.2x2.8mm_CW"
 			(at 69.85 110.49 0)
 			(hide yes)

Commit message: sch überarbeitet für neue leiste
Parts:
- added D26, D27, D28, D29, D30, D31: LED, GLR_KiCad_Library:LED_Avago_PLCC4_3.2x2.8mm_CW, symbol Device:LED
- added R5: 220, Resistor_SMD:R_2512_6332Metric_Pad1.40x3.35mm_HandSolder, symbol Device:R
- D0: renamed from D25; value 1N5822 -> STPS1L60; footprint Diode_THT:D_DO-201AD_P15.24mm_Horizontal -> Diode_SMD:D_SMA
Connections:
- net GND: now also D31.1 (K)
- net at D0.1 (K), R1.1, R2.1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: now also R5.1
- new net: D27.1 (K), D28.2 (A)
- new net: D26.1 (K), D27.2 (A)
- new net: D30.1 (K), D31.2 (A)
- new net: D26.2 (A), R5.2
- new net: D29.1 (K), D30.2 (A)
- new net: D28.1 (K), D29.2 (A)
